File: first-pcb.sch (KiCad schematic (older format))
At the start: 24 parts, among them SW1 SW_Push, U1 ATmega32U4-AU, Y1 16MHz

Commit message: V0.0.1 of the flatbrain keyboard
Parts:
- removed C1, C4, C6: 0.1uF, Capacitor_SMD:C_0805_2012Metric, symbol Device:C_Small
- removed C2, C3: 22pF, Capacitor_SMD:C_0805_2012Metric, symbol Device:C_Small
- removed C5: 1uF, Capacitor_SMD:C_0805_2012Metric, symbol Device:C_Small
- removed C7: 10uF, Diode_SMD:D_SOD-123, symbol Device:C_Small
- removed D1: D_Small, Diode_SMD:D_SOD-123, symbol Device:D_Small
- removed F1: 500mA, Fuse:Fuse_1206_3216Metric, symbol Device:Polyfuse
- removed MX1: MX-NoLED, MX_Alps_Hybrid:MX-1U-NoLED, symbol MX_Alps_Hybrid:MX-NoLED
- removed R1, R2: 22, Resistor_SMD:R_0805_2012Metric, symbol Device:R_Small
- removed R3, R4: 10k, Resistor_SMD:R_0805_2012Metric, symbol Device:R_Small
- removed U1: ATmega32U4-AU, Package_QFP:TQFP-44_10x10mm_P0.8mm, symbol MCU_Microchip_ATmega:ATmega32U4-AU
- removed USB1: Molex-0548190589, random-keyboard-parts:Molex-0548190589, symbol random-keyboard-parts:Molex-0548190589
- removed Y1: 16MHz, Crystal:Crystal_SMD_3225-4Pin_3.2x2.5mm, symbol Device:Crystal_GND24_Small
- added D10, D11, D12, D14, D15, D16, D17, D18, D19, D2, D20, D21, D22, D23, D24, D25, D26, D27, D28, D29, D3, D30, D31, D32, D33, D34, D35, D36, D37, D38, D39, D40, D41, D42, D43, D44, D5, D6, D7, D8, D9: D_Small, Diode_SMD:D_SOD-123, symbol Device:D_Small
- added J1: OLED, Connector_PinHeader_2.54mm:PinHeader_1x04_P2.54mm_Vertical, symbol corne-light-cache:Connector_Generic_Conn_01x04
- added MX10, MX11, MX12, MX14, MX15, MX16, MX17, MX18, MX19, MX2, MX20, MX21, MX22, MX23, MX24, MX25, MX26, MX27, MX28, MX29, MX3, MX30, MX31, MX32, MX33, MX34, MX35, MX36, MX37, MX38, MX39, MX40, MX41, MX42, MX43, MX44, MX5, MX6, MX7, MX8, MX9: MX-NoLED, MX_Only:MXOnly-1U-NoLED, symbol MX_Alps_Hybrid:MX-NoLED
- added U1: kbd_ProMicro, Keebio-Parts:ArduinoProMicro, symbol corne-light-cache:kbd_ProMicro
- MX1: renamed from MX2; footprint MX_Alps_Hybrid:MX-1U-NoLED -> MX_Only:MXOnly-1U-NoLED
- MX13: renamed from MX3; footprint MX_Alps_Hybrid:MX-1U-NoLED -> MX_Only:MXOnly-1U-NoLED
- MX4: footprint MX_Alps_Hybrid:MX-1U-NoLED -> MX_Only:MXOnly-1U-NoLED
- renumbered D2 to D1, D3 to D13
Connections:
- net COL0: now also MX1.1 (COL), MX25.1 (COL), MX37.1 (COL), U1.1 (TX)
- net COL1: now also MX14.1 (COL), MX2.1 (COL), MX26.1 (COL), MX38.1 (COL), U1.7 (D4); no longer MX1.1 (COL), MX4.1 (COL)
- net GND: now also J1.4 (Pin_4), U1.23 (GND), U1.3 (GND), U1.4 (GND)
- net ROW0: now also D4.1 (K), D10.1 (K), D11.1 (K), D2.1 (K), D3.1 (K), D5.1 (K), D6.1 (K), D7.1 (K), D8.1 (K), D9.1 (K), U1.20 (F4)
- net ROW1: now also D14.1 (K), D15.1 (K), D16.1 (K), D17.1 (K), D18.1 (K), D19.1 (K), D20.1 (K), D21.1 (K), D22.1 (K), D23.1 (K), U1.19 (F5); no longer D4.1 (K)
- net VCC: now also J1.3 (Pin_3), U1.21 (VCC)
- net RST: now reaches SW1.2
- net RST: now also U1.22 (RST)
- new net: D2.2 (A), MX2.2 (ROW)
- new net: D3.2 (A), MX3.2 (ROW)
- new net: D14.2 (A), MX14.2 (ROW)
- new net: D15.2 (A), MX15.2 (ROW)
- new net: D5.2 (A), MX5.2 (ROW)
- new net: D16.2 (A), MX16.2 (ROW)
- new net: D17.2 (A), MX17.2 (ROW)
- new net: D25.2 (A), MX25.2 (ROW)
- new net: D26.2 (A), MX26.2 (ROW)
- new net: D27.2 (A), MX27.2 (ROW)
- new net: D28.2 (A), MX28.2 (ROW)
- new net: D29.2 (A), MX29.2 (ROW)
- new net: D30.2 (A), MX30.2 (ROW)
- new net: D6.2 (A), MX6.2 (ROW)
- new net: D18.2 (A), MX18.2 (ROW)
- new net: D37.2 (A), MX37.2 (ROW)
- new net: D38.2 (A), MX38.2 (ROW)
- new net: D39.2 (A), MX39.2 (ROW)
- new net: D40.2 (A), MX40.2 (ROW)
- new net: D7.2 (A), MX7.2 (ROW)
- new net: D19.2 (A), MX19.2 (ROW)
- new net: D8.2 (A), MX8.2 (ROW)
- new net: D9.2 (A), MX9.2 (ROW)
- new net: D20.2 (A), MX20.2 (ROW)
- new net: D21.2 (A), MX21.2 (ROW)
- new net: D10.2 (A), MX10.2 (ROW)
- new net: D11.2 (A), MX11.2 (ROW)
- new net: D22.2 (A), MX22.2 (ROW)
- new net: D23.2 (A), MX23.2 (ROW)
- new net: D31.2 (A), MX31.2 (ROW)
- new net: D32.2 (A), MX32.2 (ROW)
- new net: D33.2 (A), MX33.2 (ROW)
- new net: D34.2 (A), MX34.2 (ROW)
- new net: D35.2 (A), MX35.2 (ROW)
- new net: D36.2 (A), MX36.2 (ROW)
- new net: D12.2 (A), MX12.2 (ROW)
- new net: D24.2 (A), MX24.2 (ROW)
- new net: D41.2 (A), MX41.2 (ROW)
- new net: D42.2 (A), MX42.2 (ROW)
- new net: D43.2 (A), MX43.2 (ROW)
- new net: D44.2 (A), MX44.2 (ROW)
- new net COL10: MX11.1 (COL), MX23.1 (COL), MX35.1 (COL), MX44.1 (COL), U1.17 (F7)
- new net COL2: MX15.1 (COL), MX27.1 (COL), MX3.1 (COL), MX39.1 (COL), U1.8 (C6)
- new net COL3: MX16.1 (COL), MX28.1 (COL), MX4.1 (COL), MX40.1 (COL), U1.9 (D7)
- new net COL4: MX17.1 (COL), MX29.1 (COL), MX41.1 (COL), MX5.1 (COL), U1.10 (E6)
- new net COL5: MX18.1 (COL), MX30.1 (COL), MX42.1 (COL), MX6.1 (COL), U1.11 (B4)
- new net COL6: MX19.1 (COL), MX31.1 (COL), MX43.1 (COL), MX7.1 (COL), U1.13 (B6)
- new net COL7: MX12.1 (COL), MX20.1 (COL), MX32.1 (COL), MX8.1 (COL), U1.14 (B2)
- new net COL8: MX21.1 (COL), MX24.1 (COL), MX33.1 (COL), MX9.1 (COL), U1.15 (B3)
- new net COL9: MX10.1 (COL), MX22.1 (COL), MX34.1 (COL), MX36.1 (COL), U1.16 (B1)
- new net ROW2: D25.1 (K), D26.1 (K), D27.1 (K), D28.1 (K), D29.1 (K), D30.1 (K), D31.1 (K), D32.1 (K), D33.1 (K), D34.1 (K), D35.1 (K), U1.18 (F6)
- new net ROW3: D12.1 (K), D24.1 (K), D36.1 (K), D37.1 (K), D38.1 (K), D39.1 (K), D40.1 (K), D41.1 (K), D42.1 (K), D43.1 (K), D44.1 (K), U1.12 (B5)
- new net SCL: J1.2 (Pin_2), U1.6 (SCL)
- new net SDA: J1.1 (Pin_1), U1.5 (SDA)
- no-connect marks 0 -> 2
Other:
- moved on the sheet: D1, D13, MX1, MX13, SW1

Commit message: Replace 1u in thumb by 1.75 and 1.5
Parts:
- MX39, MX42: footprint MX_Only:MXOnly-1U-NoLED -> MX_Only:MXOnly-1.75U-NoLED
- MX40, MX41: footprint MX_Only:MXOnly-1U-NoLED -> MX_Only:MXOnly-1.5U-NoLED
Changed lines of the file:
@@
 F 0 "MX39" H 5383 5473 60  0000 C CNN
 F 1 "MX-NoLED" H 5383 5399 20  0000 C CNN
-F 2 "MX_Only:MXOnly-1U-NoLED" H 4725 5225 60  0001 C CNN
+F 2 "MX_Only:MXOnly-1.75U-NoLED" H 4725 5225 60  0001 C CNN
 F 3 "" H 4725 5225 60  0001 C CNN
 	1    5350 5250
@@
 F 0 "MX40" H 5933 5473 60  0000 C CNN
 F 1 "MX-NoLED" H 5933 5399 20  0000 C CNN
-F 2 "MX_Only:MXOnly-1U-NoLED" H 5275 5225 60  0001 C CNN
+F 2 "MX_Only:MXOnly-1.5U-NoLED" H 5275 5225 60  0001 C CNN
 F 3 "" H 5275 5225 60  0001 C CNN
 	1    5900 5250
@@
 F 0 "MX41" H 6483 5473 60  0000 C CNN
 F 1 "MX-NoLED" H 6483 5399 20  0000 C CNN
-F 2 "MX_Only:MXOnly-1U-NoLED" H 5825 5225 60  0001 C CNN
+F 2 "MX_Only:MXOnly-1.5U-NoLED" H 5825 5225 60  0001 C CNN
 F 3 "" H 5825 5225 60  0001 C CNN
 	1    6450 5250
@@
 F 0 "MX42" H 7033 5473 60  0000 C CNN
 F 1 "MX-NoLED" H 7033 5399 20  0000 C CNN
-F 2 "MX_Only:MXOnly-1U-NoLED" H 6375 5225 60  0001 C CNN
+F 2 "MX_Only:MXOnly-1.75U-NoLED" H 6375 5225 60  0001 C CNN
 F 3 "" H 6375 5225 60  0001 C CNN
 	1    7000 5250
