File: first-pcb.kicad_pcb (KiCad board)
At the start: 2 copper layers, 91 parts, among them J1 OLED, SW1 SW_Push, U1 kbd_ProMicro

Commit message: Replace 1u in thumb by 1.75 and 1.5
Parts:
- MX39, MX42: footprint MX_Only:MXOnly-1U-NoLED -> MX_Only:MXOnly-1.75U-NoLED
- MX40, MX41: footprint MX_Only:MXOnly-1U-NoLED -> MX_Only:MXOnly-1.5U-NoLED
- moved D41 13.6 mm to (163.5, 173.0), turned to 343 degrees
- moved D42 13.5 mm to (184.2, 151.6), turned to 58 degrees
- moved D40 12.2 mm to (139.7, 165.1), turned to 107 degrees
- moved D39 2.68 mm to (123.0, 150.8)
- turned MX39 to 32 degrees
- turned MX40 to 17 degrees
- turned MX41 to 343 degrees
- turned MX42 to 328 degrees
Routing:
- net COL5: track 147.7 -> 163.7 mm
- net COL3: track 179.1 -> 192.3 mm
- net COL4: track 170.2 -> 178.2 mm
- net Net-(D22-Pad2): track 0.00 -> 6.65 mm
- net Net-(D41-Pad2): track 7.21 -> 11.5 mm
- net Net-(D39-Pad2): track 7.58 -> 11.4 mm
- net Net-(D42-Pad2): track 7.22 -> 9.38 mm
- net COL2: track 195.0 -> 196.4 mm
- net COL1: track 212.0 -> 213.3 mm
- net Net-(D40-Pad2): track 7.15 -> 8.42 mm
- net ROW3: track 670.3 -> 671.4 mm

Commit message: Perfect alignement
Parts:
- moved D18 5.35 mm to (134.1, 113.9)
- moved D40 5.35 mm to (141.1, 170.2)
- moved D1 5.35 mm to (54.5, 60.4)
- moved D13 5.35 mm to (45.3, 76.9)
- moved D14 5.35 mm to (62.4, 86.1)
- moved D15 5.35 mm to (84.9, 83.8)
- moved D16 5.35 mm to (104.6, 87.1)
- moved D17 5.35 mm to (118.3, 102.8)
- moved D2 5.35 mm to (71.4, 69.2)
- moved D25 5.35 mm to (36.6, 93.2)
- moved D26 5.35 mm to (53.5, 102.9)
- moved D27 5.35 mm to (75.8, 101.2)
- moved D28 5.35 mm to (95.7, 105.0)
- moved D38 5.35 mm to (106.1, 145.1)
- moved D39 5.35 mm to (124.5, 156.0)
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Routing:
- net ROW3: track 671.4 -> 217.0 mm
- net ROW0: track 559.8 -> 215.9 mm
- net ROW2: track 531.8 -> 211.4 mm
- net ROW1: track 551.4 -> 272.9 mm
- net COL7: track 248.7 -> 41.1 mm
- net COL8: track 222.0 -> 41.0 mm
- net COL9: track 202.3 -> 41.0 mm
- net COL4: track 178.2 -> 46.0 mm
- net COL5: track 163.7 -> 45.8 mm
- net COL0: track 180.5 -> 73.9 mm
- net GND: track 88.5 -> 0.00 mm
- net COL1: track 213.3 -> 125.6 mm
- net COL10: track 141.9 -> 61.5 mm
- net VCC: track 76.8 -> 0.00 mm
- net SDA: track 65.4 -> 0.00 mm
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
Commit message: routing corrected
Parts:
- moved J1 6.35 mm to (153.0, 115.2)
Routing:
- net ROW3: track 217.0 -> 662.4 mm
- net ROW0: track 215.9 -> 558.6 mm
- net ROW2: track 211.4 -> 521.1 mm
- net ROW1: track 272.9 -> 538.9 mm
- net COL7: track 41.1 -> 232.6 mm
- net COL8: track 41.0 -> 207.6 mm
- net COL9: track 41.0 -> 189.7 mm
- net COL5: track 45.8 -> 179.8 mm
- net COL4: track 46.0 -> 179.1 mm
- net COL0: track 73.9 -> 195.8 mm
- net COL1: track 125.6 -> 214.6 mm
- net GND: track 0.00 -> 88.8 mm
- net COL10: track 61.5 -> 149.1 mm
- net VCC: track 0.00 -> 69.9 mm
- net COL2: track 131.1 -> 195.7 mm
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
Commit message: realign + outline
Parts:
- moved MX24 0.06 mm to (259.9, 73.4)
- moved MX35 0.06 mm to (252.0, 99.1)
- moved MX44 0.06 mm to (260.9, 115.9)
- moved MX36 0.06 mm to (268.8, 90.2)
Routing:
- net COL9: track 189.7 -> 193.2 mm
- net COL7: track 232.6 -> 234.6 mm
- net COL8: track 207.6 -> 209.0 mm
- net ROW1: track 538.9 -> 539.6 mm
Other:
- board outline added: 267 x 144.4 mm

Commit message: final design
Parts:
- moved U1 0.16 mm to (149.2, 61.4)
- moved MX33 0.13 mm to (210.0, 101.2)
- moved MX9 0.13 mm to (192.1, 67.6)
- moved MX21 0.13 mm to (201.0, 84.4)
- moved MX8 0.13 mm to (178.3, 82.2)
- moved MX20 0.13 mm to (187.2, 99.0)
- moved MX22 0.12 mm to (220.6, 80.7)
- moved MX34 0.12 mm to (229.6, 97.5)
- moved MX10 0.12 mm to (211.7, 63.9)
- moved MX32 0.11 mm to (196.2, 115.9)
Routing:
- net ROW3: track 662.7 -> 667.6 mm
Other:
- board size 267 x 144.4 mm -> 272.2 x 143 mm

Commit message: first revision is over
Parts:
- moved D24 9.44 mm to (262.2, 77.8), turned to 28 degrees
- moved D12 8.73 mm to (253.5, 60.8), turned to 28 degrees
- moved D36 8.68 mm to (271.4, 94.5), turned to 28 degrees
Routing:
- net ROW3: track 667.6 -> 647.0 mm
- net Net-(D12-Pad2): track 6.38 -> 10.9 mm
- net Net-(D24-Pad2): track 6.56 -> 11.0 mm
- net Net-(D36-Pad2): track 6.54 -> 10.9 mm
Other:
- outline, holes or cut-outs redrawn

Commit message: New routing to use less pin
Parts:
- U1: moved to B.Cu
- moved MX12 10.2 mm to (250.0, 46.4)
- moved MX17 10.2 mm to (110.2, 88.9)
- moved D2 10.2 mm to (70.4, 59.1)
- moved D32 10.2 mm to (202.1, 101.9)
- moved D20 10.2 mm to (193.4, 85.1)
- moved D35 10.2 mm to (258.0, 85.2)
- moved MX40 10.2 mm to (130.9, 162.6)
- moved D27 10.2 mm to (74.8, 91.1)
- moved MX33 10.2 mm to (209.0, 91.1)
- moved D29 10.2 mm to (108.1, 109.4)
- moved D33 10.2 mm to (215.9, 87.2)
- moved MX25 10.2 mm to (28.6, 80.1)
- moved MX27 10.2 mm to (67.9, 87.4)
- moved D16 10.2 mm to (103.6, 77.0)
- moved MX26 10.2 mm to (45.5, 89.0)
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Connections:
- D10 pad 1: ROW0 -> ROW4
- D11 pad 1: ROW0 -> ROW4
- D12 pad 1: ROW3 -> ROW4
- D19 pad 1: ROW1 -> ROW5
- D20 pad 1: ROW1 -> ROW5
- D21 pad 1: ROW1 -> ROW5
- D22 pad 1: ROW1 -> ROW5
- D23 pad 1: ROW1 -> ROW5
- D24 pad 1: ROW3 -> ROW5
- D31 pad 1: ROW2 -> ROW6
- D32 pad 1: ROW2 -> ROW6
- D33 pad 1: ROW2 -> ROW6
- D34 pad 1: ROW2 -> ROW6
- D35 pad 1: ROW2 -> ROW6
- D36 pad 1: ROW3 -> ROW6
- D41 pad 1: ROW3 -> ROW7
- D42 pad 1: ROW3 -> ROW7
- D43 pad 1: ROW3 -> ROW7
- D44 pad 1: ROW3 -> ROW7
- D7 pad 1: ROW0 -> ROW4
- D8 pad 1: ROW0 -> ROW4
- D9 pad 1: ROW0 -> ROW4
- MX10 pad 1: COL9 -> COL2
- MX11 pad 1: COL10 -> COL1
- MX12 pad 1: COL7 -> COL0
- MX19 pad 1: COL6 -> COL5
- MX20 pad 1: COL7 -> COL4
- MX21 pad 1: COL8 -> COL3
- MX22 pad 1: COL9 -> COL2
- MX23 pad 1: COL10 -> COL1
- MX24 pad 1: COL8 -> COL0
- MX31 pad 1: COL6 -> COL5
- MX32 pad 1: COL7 -> COL4
- MX33 pad 1: COL8 -> COL3
- MX34 pad 1: COL9 -> COL2
- MX35 pad 1: COL10 -> COL1
- MX36 pad 1: COL9 -> COL0
- MX37 pad 1: COL0 -> COL1
- MX38 pad 1: COL1 -> COL3
- MX39 pad 1: COL2 -> COL4
- MX40 pad 1: COL3 -> COL5
- MX41 pad 1: COL4 -> COL5
- MX42 pad 1: COL5 -> COL4
- MX43 pad 1: COL6 -> COL3
- MX44 pad 1: COL10 -> COL1
- MX7 pad 1: COL6 -> COL5
- MX8 pad 1: COL7 -> COL4
- MX9 pad 1: COL8 -> COL3
- U1 pad 1: COL0 -> Net-(U1-Pad1)
- U1 pad 10: COL4 -> ROW7
- U1 pad 11: COL5 -> ROW2
- U1 pad 13: COL6 -> COL5
- U1 pad 14: COL7 -> COL4
- U1 pad 15: COL8 -> COL3
- U1 pad 16: COL9 -> COL2
- U1 pad 17: COL10 -> COL1
- U1 pad 18: ROW2 -> COL0
- U1 pad 19: ROW1 -> ROW0
- U1 pad 20: ROW0 -> ROW1
- U1 pad 7: COL1 -> ROW4
- U1 pad 8: COL2 -> ROW5
- U1 pad 9: COL3 -> ROW6
Routing:
- net ROW0: track 558.6 -> 154.7 mm
- net COL0: track 195.8 -> 585.0 mm
- net ROW3: track 647.0 -> 259.8 mm
- net ROW1: track 539.6 -> 183.1 mm
- net ROW2: track 521.4 -> 188.4 mm
- net COL1: track 214.6 -> 520.9 mm
- net ROW7: track 0.00 -> 289.5 mm
- net COL7: track 235.0 -> 0.00 mm
- net COL8: track 209.0 -> 0.00 mm
- net COL2: track 195.7 -> 398.6 mm
- net COL9: track 193.2 -> 0.00 mm
- net ROW6: track 0.00 -> 191.5 mm
- net ROW5: track 0.00 -> 175.0 mm
- net COL3: track 191.2 -> 349.6 mm
- net COL10: track 149.1 -> 0.00 mm
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
Commit message: Routing the LED
Parts:
- added LED1: WS2812B, LED_SMD:LED_WS2812B_PLCC4_5.0x5.0mm_P3.2mm, B.Cu at (92.5, 61.4)
- added LED10: WS2812B, LED_SMD:LED_WS2812B_PLCC4_5.0x5.0mm_P3.2mm, B.Cu at (148.2, 48.4)
- added LED2: WS2812B, LED_SMD:LED_WS2812B_PLCC4_5.0x5.0mm_P3.2mm, B.Cu at (50.5, 59.3)
- added LED3: WS2812B, LED_SMD:LED_WS2812B_PLCC4_5.0x5.0mm_P3.2mm, B.Cu at (32.6, 92.9)
- added LED4: WS2812B, LED_SMD:LED_WS2812B_PLCC4_5.0x5.0mm_P3.2mm, B.Cu at (67.9, 113.6)
- added LED5: WS2812B, LED_SMD:LED_WS2812B_PLCC4_5.0x5.0mm_P3.2mm, B.Cu at (148.2, 152.1)
- added LED6: WS2812B, LED_SMD:LED_WS2812B_PLCC4_5.0x5.0mm_P3.2mm, B.Cu at (228.6, 113.6)
- added LED7: WS2812B, LED_SMD:LED_WS2812B_PLCC4_5.0x5.0mm_P3.2mm, B.Cu at (263.9, 92.9)
- added LED8: WS2812B, LED_SMD:LED_WS2812B_PLCC4_5.0x5.0mm_P3.2mm, B.Cu at (246.0, 59.3)
- added LED9: WS2812B, LED_SMD:LED_WS2812B_PLCC4_5.0x5.0mm_P3.2mm, B.Cu at (204.0, 61.4)
- moved D3 11.4 mm to (81.8, 60.3), turned to 152 degrees
Connections:
- U1 pad 1: Net-(U1-Pad1) -> LED
Routing:
- net VCC: track 66.4 -> 691.3 mm, vias 0 -> 3
- net GND: track 90.9 -> 646.5 mm, vias 0 -> 1
- net Net-(LED5-Pad2): track 0.00 -> 114.8 mm
- net Net-(LED4-Pad2): track 0.00 -> 109.7 mm
- net Net-(LED10-Pad4): track 0.00 -> 83.8 mm
- net Net-(LED1-Pad2): track 0.00 -> 82.5 mm
- net LED: track 0.00 -> 77.7 mm
- net Net-(LED7-Pad2): track 0.00 -> 64.0 mm
- net Net-(LED6-Pad2): track 0.00 -> 54.7 mm
- net Net-(LED3-Pad2): track 0.00 -> 53.8 mm
- net Net-(LED8-Pad2): track 0.00 -> 44.7 mm
- net Net-(LED2-Pad2): track 0.00 -> 44.4 mm
- net Net-(D3-Pad2): track 6.75 -> 14.7 mm
- net ROW0: track 154.7 -> 155.5 mm
