File: first-pcb.kicad_pcb (KiCad board)
At the start: 2 copper layers, 272.2 x 143 mm, 91 parts, among them J1 OLED, SW1 SW_Push, U1 kbd_ProMicro

Commit message: Version 0.1.1 (#2)
* New routing to use less pin

* Add LED on the schema

* Routing the LED

* Change the silks to display switch info

* add the plate dxf file

* Rename contour in bottom
Parts:
- added LED1: WS2812B, LED_SMD:LED_WS2812B_PLCC4_5.0x5.0mm_P3.2mm, B.Cu at (92.5, 61.4)
- added LED10: WS2812B, LED_SMD:LED_WS2812B_PLCC4_5.0x5.0mm_P3.2mm, B.Cu at (148.2, 48.4)
- added LED2: WS2812B, LED_SMD:LED_WS2812B_PLCC4_5.0x5.0mm_P3.2mm, B.Cu at (50.5, 59.3)
- added LED3: WS2812B, LED_SMD:LED_WS2812B_PLCC4_5.0x5.0mm_P3.2mm, B.Cu at (32.6, 92.9)
- added LED4: WS2812B, LED_SMD:LED_WS2812B_PLCC4_5.0x5.0mm_P3.2mm, B.Cu at (67.9, 113.6)
- added LED5: WS2812B, LED_SMD:LED_WS2812B_PLCC4_5.0x5.0mm_P3.2mm, B.Cu at (148.2, 152.1)
- added LED6: WS2812B, LED_SMD:LED_WS2812B_PLCC4_5.0x5.0mm_P3.2mm, B.Cu at (228.6, 113.6)
- added LED7: WS2812B, LED_SMD:LED_WS2812B_PLCC4_5.0x5.0mm_P3.2mm, B.Cu at (263.9, 92.9)
- added LED8: WS2812B, LED_SMD:LED_WS2812B_PLCC4_5.0x5.0mm_P3.2mm, B.Cu at (246.0, 59.3)
- added LED9: WS2812B, LED_SMD:LED_WS2812B_PLCC4_5.0x5.0mm_P3.2mm, B.Cu at (204.0, 61.4)
- MX1, MX10, MX11, MX12, MX13, MX14, MX15, MX16, MX17, MX18, MX19, MX2, MX20, MX21, MX22, MX23, MX24, MX25, MX26, MX27, MX28, MX29, MX3, MX30, MX31, MX32, MX33, MX34, MX35, MX36, MX37, MX38, MX4, MX43, MX44, MX5, MX6, MX7, MX8, MX9: value MX-NoLED -> 1U
- MX39, MX42: value MX-NoLED -> 1.75U
- MX40, MX41: value MX-NoLED -> 1.5U
- U1: moved to B.Cu
- moved D3 13.7 mm to (81.8, 60.3), turned to 152 degrees
- moved MX12 10.2 mm to (250.0, 46.4)
- moved MX17 10.2 mm to (110.2, 88.9)
- moved D2 10.2 mm to (70.4, 59.1)
- moved D35 10.2 mm to (258.0, 85.2)
- moved D20 10.2 mm to (193.4, 85.1)
- moved D32 10.2 mm to (202.1, 101.9)
- moved MX40 10.2 mm to (130.9, 162.6)
- moved D27 10.2 mm to (74.8, 91.1)
- moved D29 10.2 mm to (108.1, 109.4)
- moved MX33 10.2 mm to (209.0, 91.1)
- moved MX25 10.2 mm to (28.6, 80.1)
- moved MX27 10.2 mm to (67.9, 87.4)
- moved D16 10.2 mm to (103.6, 77.0)
- moved MX26 10.2 mm to (45.5, 89.0)
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Connections:
- D10 pad 1: ROW0 -> ROW4
- D11 pad 1: ROW0 -> ROW4
- D12 pad 1: ROW3 -> ROW4
- D19 pad 1: ROW1 -> ROW5
- D20 pad 1: ROW1 -> ROW5
- D21 pad 1: ROW1 -> ROW5
- D22 pad 1: ROW1 -> ROW5
- D23 pad 1: ROW1 -> ROW5
- D24 pad 1: ROW3 -> ROW5
- D31 pad 1: ROW2 -> ROW6
- D32 pad 1: ROW2 -> ROW6
- D33 pad 1: ROW2 -> ROW6
- D34 pad 1: ROW2 -> ROW6
- D35 pad 1: ROW2 -> ROW6
- D36 pad 1: ROW3 -> ROW6
- D41 pad 1: ROW3 -> ROW7
- D42 pad 1: ROW3 -> ROW7
- D43 pad 1: ROW3 -> ROW7
- D44 pad 1: ROW3 -> ROW7
- D7 pad 1: ROW0 -> ROW4
- D8 pad 1: ROW0 -> ROW4
- D9 pad 1: ROW0 -> ROW4
- MX10 pad 1: COL9 -> COL2
- MX11 pad 1: COL10 -> COL1
- MX12 pad 1: COL7 -> COL0
- MX19 pad 1: COL6 -> COL5
- MX20 pad 1: COL7 -> COL4
- MX21 pad 1: COL8 -> COL3
- MX22 pad 1: COL9 -> COL2
- MX23 pad 1: COL10 -> COL1
- MX24 pad 1: COL8 -> COL0
- MX31 pad 1: COL6 -> COL5
- MX32 pad 1: COL7 -> COL4
- MX33 pad 1: COL8 -> COL3
- MX34 pad 1: COL9 -> COL2
- MX35 pad 1: COL10 -> COL1
- MX36 pad 1: COL9 -> COL0
- MX37 pad 1: COL0 -> COL1
- MX38 pad 1: COL1 -> COL3
- MX39 pad 1: COL2 -> COL4
- MX40 pad 1: COL3 -> COL5
- MX41 pad 1: COL4 -> COL5
- MX42 pad 1: COL5 -> COL4
- MX43 pad 1: COL6 -> COL3
- MX44 pad 1: COL10 -> COL1
- MX7 pad 1: COL6 -> COL5
- MX8 pad 1: COL7 -> COL4
- MX9 pad 1: COL8 -> COL3
- U1 pad 1: COL0 -> LED
- U1 pad 10: COL4 -> ROW7
- U1 pad 11: COL5 -> ROW2
- U1 pad 13: COL6 -> COL5
- U1 pad 14: COL7 -> COL4
- U1 pad 15: COL8 -> COL3
- U1 pad 16: COL9 -> COL2
- U1 pad 17: COL10 -> COL1
- U1 pad 18: ROW2 -> COL0
- U1 pad 19: ROW1 -> ROW0
- U1 pad 20: ROW0 -> ROW1
- U1 pad 7: COL1 -> ROW4
- U1 pad 8: COL2 -> ROW5
- U1 pad 9: COL3 -> ROW6
Routing:
- net VCC: track 69.9 -> 691.3 mm, vias 0 -> 3
- net GND: track 89.1 -> 646.4 mm, vias 0 -> 1
- net ROW0: track 558.6 -> 155.5 mm
- net COL0: track 195.8 -> 585.0 mm
- net ROW3: track 647.0 -> 259.8 mm
- net ROW1: track 539.6 -> 183.1 mm
- net ROW2: track 521.4 -> 188.4 mm
- net COL1: track 214.6 -> 520.9 mm
- net ROW7: track 0.00 -> 289.5 mm
- net COL7: track 235.0 -> 0.00 mm
- net COL8: track 209.0 -> 0.00 mm
- net COL2: track 195.7 -> 398.6 mm
- net COL9: track 193.2 -> 0.00 mm
- net ROW6: track 0.00 -> 191.5 mm
- net ROW5: track 0.00 -> 175.0 mm
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Other:
- board text added: "Designed by louckousse"
- board text added: "JLCJLCJLCJLC"
