File: first-pcb.kicad_pcb (KiCad board)
At the start: 2 copper layers, 272.2 x 143 mm, 101 parts, among them J1 OLED, SW1 SW_Push, U1 kbd_ProMicro

Commit message: Change the silks to display switch info
Parts:
- MX1, MX10, MX11, MX12, MX13, MX14, MX15, MX16, MX17, MX18, MX19, MX2, MX20, MX21, MX22, MX23, MX24, MX25, MX26, MX27, MX28, MX29, MX3, MX30, MX31, MX32, MX33, MX34, MX35, MX36, MX37, MX38, MX4, MX43, MX44, MX5, MX6, MX7, MX8, MX9: value MX-NoLED -> 1U
- MX39, MX42: value MX-NoLED -> 1.75U
- MX40, MX41: value MX-NoLED -> 1.5U
Other:
- board text added: "Designed by louckousse"
- board text added: "JLCJLCJLCJLC"

Commit message: Replace smd diode with hybrid
Parts:
- D1, D10, D11, D12, D13, D14, D15, D16, D17, D18, D19, D2, D20, D21, D22, D23, D24, D25, D26, D27, D28, D29, D3, D30, D31, D32, D33, D34, D35, D36, D37, D38, D39, D4, D40, D41, D42, D43, D44, D5, D6, D7, D8, D9: footprint Diode_SMD:D_SOD-123 -> Keebio-Parts:Diode-Hybrid-Back; moved to F.Cu
- moved D40 20.6 mm to (139.1, 139.6), turned to 287 degrees
- moved D41 17.3 mm to (163.7, 150.7), turned to 163 degrees
- moved MX34 15.9 mm to (227.9, 71.5)
- moved MX11 15.9 mm to (232.4, 39.4)
- moved MX31 15.9 mm to (178.8, 100.9)
- moved D21 15.9 mm to (206.3, 54.5), turned to 298 degrees
- moved MX27 15.9 mm to (67.2, 71.5)
- moved MX28 15.9 mm to (86.8, 75.1)
- moved MX43 15.9 mm to (196.3, 113.6)
- moved D17 15.9 mm to (116.6, 76.7), turned to 242 degrees
- moved D23 15.9 mm to (248.4, 52.5), turned to 298 degrees
- moved D7 15.9 mm to (167.8, 63.6), turned to 298 degrees
- moved LED5 15.9 mm to (147.5, 136.2)
- moved MX32 15.9 mm to (194.5, 89.8)
- moved MX44 15.9 mm to (259.2, 89.9)
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Routing:
- net GND: track 646.4 -> 677.6 mm
- net COL0: track 585.0 -> 604.3 mm
- net Net-(LED6-Pad2): track 54.7 -> 69.4 mm
- net VCC: track 691.3 -> 705.9 mm
- net Net-(LED2-Pad2): track 44.4 -> 57.9 mm
- net COL2: track 398.6 -> 410.2 mm
- net Net-(LED10-Pad4): track 83.8 -> 91.5 mm
- net COL1: track 520.9 -> 526.5 mm
- net ROW3: track 259.8 -> 255.3 mm
- net COL5: track 232.0 -> 235.8 mm
- net Net-(LED1-Pad2): track 82.5 -> 84.2 mm
- net Net-(D41-Pad2): track 11.3 -> 9.97 mm
- net ROW0: track 155.5 -> 156.8 mm
- net ROW4: track 141.4 -> 142.7 mm
- net ROW1: track 183.1 -> 184.3 mm
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