File: flatbrain.kicad_pcb (KiCad board)
At the start: 2 copper layers, 272.2 x 143 mm, 101 parts, among them J1 OLED, SW1 SW_Push, U1 kbd_ProMicro

Commit message: diode placement
Parts:
- moved D39 10.6 mm to (127.9, 120.5), turned to 302 degrees
- moved D36 9.81 mm to (260.1, 67.9), turned to 298 degrees
- moved D12 9.76 mm to (242.2, 34.2), turned to 298 degrees
- moved D24 9.60 mm to (251.2, 51.0), turned to 298 degrees
- moved D41 9.24 mm to (173.0, 149.0), turned to 253 degrees
- moved D40 4.69 mm to (138.4, 144.2)
- moved D42 2.51 mm to (181.7, 129.2)
- moved D16 1.00 mm to (103.3, 62.1)
- moved D5 0.77 mm to (126.0, 59.9)
- moved D25 0.75 mm to (35.5, 67.9)
- moved D15 0.68 mm to (83.7, 58.4)
- moved D13 0.64 mm to (44.4, 51.0)
- moved D9 0.62 mm to (197.9, 37.5)
- moved D3 0.62 mm to (81.5, 45.0)
- moved D7 0.52 mm to (168.5, 63.2)
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Routing:
- net Net-(LED10-Pad4): track 91.5 -> 106.5 mm
- net COL0: track 604.3 -> 615.4 mm
- net Net-(D24-Pad2): track 10.5 -> 19.9 mm
- net ROW4: track 142.7 -> 134.1 mm
- net ROW2: track 189.5 -> 181.3 mm
- net ROW0: track 156.8 -> 149.3 mm
- net ROW5: track 175.0 -> 168.8 mm
- net ROW1: track 184.3 -> 178.2 mm
- net ROW3: track 255.3 -> 249.8 mm
- net Net-(D39-Pad2): track 11.2 -> 6.20 mm
- net COL3: track 350.6 -> 355.6 mm
- net COL1: track 526.5 -> 531.0 mm
- net COL2: track 410.2 -> 414.7 mm
- net VCC: track 705.9 -> 701.8 mm
- net Net-(D41-Pad2): track 9.97 -> 6.20 mm
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
Commit message: Correct leds connection
Parts:
- MX1, MX10, MX11, MX12, MX13, MX14, MX15, MX16, MX17, MX18, MX19, MX2, MX20, MX21, MX22, MX23, MX24, MX25, MX26, MX27, MX28, MX29, MX3, MX30, MX31, MX32, MX33, MX34, MX35, MX36, MX37, MX38, MX4, MX43, MX44, MX5, MX6, MX7, MX8, MX9: value 1U -> MX-NoLED; footprint MX_Only:MXOnly-1U-NoLED -> parts:mx_1u
- MX39, MX42: value 1.75U -> MX-NoLED; footprint MX_Only:MXOnly-1.75U-NoLED -> parts:mx_175u
- MX40, MX41: value 1.5U -> MX-NoLED; footprint MX_Only:MXOnly-1.5U-NoLED -> parts:mx_15u
Connections:
- LED1 pad 1: GND -> VCC
- LED1 pad 3: VCC -> GND
- LED10 pad 1: GND -> VCC
- LED10 pad 3: VCC -> GND
- LED2 pad 1: GND -> VCC
- LED2 pad 3: VCC -> GND
- LED3 pad 1: GND -> VCC
- LED3 pad 3: VCC -> GND
- LED4 pad 1: GND -> VCC
- LED4 pad 3: VCC -> GND
- LED5 pad 1: GND -> VCC
- LED5 pad 3: VCC -> GND
- LED6 pad 1: GND -> VCC
- LED6 pad 3: VCC -> GND
- LED7 pad 1: GND -> VCC
- LED7 pad 3: VCC -> GND
- LED8 pad 1: GND -> VCC
- LED8 pad 3: VCC -> GND
- LED9 pad 1: GND -> VCC
- LED9 pad 3: VCC -> GND
Routing:
- net GND: track 678.2 -> 637.6 mm, vias 1 -> 2
- net VCC: track 701.8 -> 716.4 mm
- net Net-(D24-Pad2): track 19.9 -> 11.3 mm
- net Net-(LED5-Pad2): track 117.1 -> 121.7 mm
- net Net-(D44-Pad2): track 6.90 -> 6.20 mm
- net ROW5: track 168.8 -> 168.1 mm

Commit message: Move lowest pinky keys to thumb cluster
Parts:
- moved D44 161.2 mm to (140.1, 185.4), turned to 270 degrees
- moved MX44 146.7 mm to (148.3, 185.4), turned to 0 degrees
- moved MX36 126.2 mm to (212.8, 177.8), turned to 0 degrees
- moved LED7 125.8 mm to (203.3, 187.3), turned to 332 degrees
- moved D36 123.2 mm to (204.6, 177.8), turned to 270 degrees
- moved D35 122.2 mm to (202.0, 177.8), turned to 270 degrees
- moved MX24 120.5 mm to (212.8, 158.7), turned to 0 degrees
- moved MX35 119.3 mm to (193.8, 177.8), turned to 0 degrees
- moved D24 117.3 mm to (204.6, 158.7), turned to 270 degrees
- moved D23 116.4 mm to (202.0, 158.7), turned to 270 degrees
- moved MX12 115.3 mm to (212.8, 139.7), turned to 0 degrees
- moved LED8 114.1 mm to (203.3, 149.2), turned to 332 degrees
- moved MX23 113.2 mm to (193.8, 158.7), turned to 0 degrees
- moved LED6 112.6 mm to (162.4, 189.0), turned to 152 degrees
- moved D12 112.0 mm to (204.6, 139.7), turned to 270 degrees
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Routing:
- net ROW3: track 249.8 -> 173.1 mm
- net COL0: track 615.4 -> 576.5 mm
- net COL1: track 531.0 -> 503.8 mm
- net Net-(D44-Pad2): track 6.20 -> 17.5 mm
- net Net-(LED5-Pad2): track 121.7 -> 116.4 mm
Other:
- board size 272.2 x 143 mm -> 245.6 x 188.5 mm

Commit message: Work in progress:
Replace pro-micro with Elite-C
Add 2 rotary encoders
Parts:
- added D41: D_Small, Keebio-Parts:Diode-Hybrid-Back, F.Cu at (177.5, 17.3)
- added D42: D_Small, Keebio-Parts:Diode-Hybrid-Back, F.Cu at (194.4, 20.8)
- added JP1: Jumper_NO_Small, Jumper:SolderJumper-2_P1.3mm_Open_Pad1.0x1.5mm, F.Cu at (187.8, 14.6)
- added JP2: Jumper_NO_Small, Jumper:SolderJumper-2_P1.3mm_Open_Pad1.0x1.5mm, F.Cu at (209.7, 17.0)
- added JP3: Jumper_NO_Small, Jumper:SolderJumper-2_P1.3mm_Open_Pad1.0x1.5mm, F.Cu at (200.0, 14.0)
- added SW41: Rotary_Encoder_Switch, parts:rotary_x_mx, F.Cu at (164.8, 1.02)
- added SW42: Rotary_Encoder_Switch, parts:rotary_x_mx, F.Cu at (196.0, -2.79)
- U1: value kbd_ProMicro -> Elite-C; footprint Keebio-Parts:ArduinoProMicro -> Keebio-Parts:Elite-C
- moved MX36 126.1 mm to (267.4, 64.1), turned to 28 degrees
- moved LED7 125.7 mm to (263.5, 77.0), turned to 0 degrees
- moved D36 123.1 mm to (260.1, 68.0), turned to 298 degrees
- moved D35 122.1 mm to (257.9, 69.2), turned to 298 degrees
- moved MX24 120.4 mm to (258.5, 47.3), turned to 28 degrees
- moved MX35 119.1 mm to (250.6, 73.1), turned to 28 degrees
- moved D24 117.2 mm to (251.2, 51.2), turned to 298 degrees
- moved D23 116.3 mm to (249.0, 52.4), turned to 298 degrees
- moved MX12 115.2 mm to (249.5, 30.5), turned to 28 degrees
- moved LED8 114.0 mm to (245.6, 43.4), turned to 0 degrees
- moved MX23 113.1 mm to (241.7, 56.2), turned to 28 degrees
- moved LED6 112.5 mm to (228.2, 97.7), turned to 180 degrees
- moved D12 111.9 mm to (242.3, 34.4), turned to 298 degrees
- moved D34 111.4 mm to (235.5, 67.6), turned to 298 degrees
- moved D11 110.8 mm to (240.0, 35.6), turned to 298 degrees
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- renumbered D41 to D43, D42 to D44, D43 to D45, D44 to D46, MX41 to MX43, MX42 to MX44, MX43 to MX45, MX44 to MX46
Connections:
- D10 pad 1: ROW4 -> ROW0
- D11 pad 1: ROW4 -> ROW0
- D12 pad 1: ROW4 -> ROW0
- D19 pad 1: ROW5 -> ROW1
- D20 pad 1: ROW5 -> ROW1
- D21 pad 1: ROW5 -> ROW1
- D22 pad 1: ROW5 -> ROW1
- D23 pad 1: ROW5 -> ROW1
- D24 pad 1: ROW5 -> ROW1
- D31 pad 1: ROW6 -> ROW2
- D32 pad 1: ROW6 -> ROW2
- D33 pad 1: ROW6 -> ROW2
- D34 pad 1: ROW6 -> ROW2
- D35 pad 1: ROW6 -> ROW2
- D36 pad 1: ROW6 -> ROW2
- D43 pad 1: ROW7 -> ROW3
- D44 pad 1: ROW7 -> ROW3
- D45 pad 1: ROW7 -> ROW3
- D46 pad 1: ROW7 -> ROW3
- D7 pad 1: ROW4 -> ROW0
- D8 pad 1: ROW4 -> ROW0
- D9 pad 1: ROW4 -> ROW0
- MX10 pad 1: COL2 -> COL9
- MX11 pad 1: COL1 -> COL10
- MX12 pad 1: COL0 -> COL11
- MX19 pad 1: COL5 -> COL6
- MX20 pad 1: COL4 -> COL7
- MX21 pad 1: COL3 -> COL8
- MX22 pad 1: COL2 -> COL9
- MX23 pad 1: COL1 -> COL10
- MX24 pad 1: COL0 -> COL11
- MX31 pad 1: COL5 -> COL6
- MX32 pad 1: COL4 -> COL7
- MX33 pad 1: COL3 -> COL8
- MX34 pad 1: COL2 -> COL9
- MX35 pad 1: COL1 -> COL10
- MX36 pad 1: COL0 -> COL11
- MX38 pad 1: COL3 -> COL2
- MX39 pad 1: COL4 -> COL3
- MX40 pad 1: COL5 -> COL4
- MX43 pad 1: COL5 -> COL7
- MX44 pad 1: COL4 -> COL8
- MX45 pad 1: COL3 -> COL9
- MX46 pad 1: COL1 -> COL10
- MX7 pad 1: COL5 -> COL6
- MX8 pad 1: COL4 -> COL7
- MX9 pad 1: COL3 -> COL8
- U1 pad 1: LED -> Net-(JP2-Pad2)
- U1 pad 10: ROW7 -> COL3
- U1 pad 11: ROW2 -> COL4
- U1 pad 12: ROW3 -> COL5
- U1 pad 13: COL5 -> COL6
- U1 pad 14: COL4 -> COL7
- U1 pad 15: COL3 -> COL8
- U1 pad 16: COL2 -> COL9
- U1 pad 17: COL1 -> COL10
- U1 pad 18: COL0 -> COL11
- U1 pad 19: ROW0 -> ROW3
- U1 pad 2: Net-(U1-Pad2) -> ROW1
- U1 pad 20: ROW1 -> ROW2
- U1 pad 7: ROW4 -> COL0
- U1 pad 8: ROW5 -> COL1
- U1 pad 9: ROW6 -> COL2
Routing:
- net COL1: track 503.8 -> 460.2 mm
- net COL0: track 576.5 -> 537.9 mm
- net ROW7: track 292.1 -> 257.4 mm
- net COL2: track 414.7 -> 424.8 mm
- net Net-(D46-Pad2): track 17.5 -> 11.3 mm
Other:
- board size 245.6 x 188.5 mm -> 272.2 x 143 mm

Commit message: Reroute left half
Parts:
- JP1, JP2, JP3: moved to B.Cu
- MX39, MX44: footprint parts:mx_175u -> parts:mx_1u
- MX40, MX43: footprint parts:mx_15u -> parts:mx_1u
- moved LED3 238.6 mm to (270.6, 84.3), turned to 28 degrees
- moved LED7 236.1 mm to (27.5, 84.3), turned to 332 degrees
- moved LED2 204.4 mm to (254.4, 40.7), turned to 28 degrees
- moved LED8 194.4 mm to (51.3, 46.7), turned to 332 degrees
- moved LED4 166.7 mm to (234.1, 101.8), turned to 208 degrees
- moved LED6 144.4 mm to (84.9, 115.6), turned to 332 degrees
- moved SW42 129.3 mm to (167.1, 123.2), turned to 53 degrees
- moved SW41 126.2 mm to (130.5, 122.4), turned to 307 degrees
- moved Dn 119.4 mm to (135.5, 129.0), turned to 217 degrees
- moved D42 115.7 mm to (162.4, 132.0)
- moved LED1 108.6 mm to (200.5, 38.3), turned to 28 degrees
- moved LED9 104.4 mm to (99.5, 37.3), turned to 152 degrees
- moved JP1 57.3 mm to (135.0, 36.7), turned to 180 degrees
- moved JP2 50.5 mm to (163.2, 36.7), turned to 180 degrees
- moved JP3 44.7 mm to (163.2, 39.2), turned to 180 degrees
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- renumbered D41 to Dn
Connections:
- U1 pad 10: COL3 -> COL9
- U1 pad 11: COL4 -> COL10
- U1 pad 12: COL5 -> COL11
- U1 pad 13: COL6 -> COL5
- U1 pad 14: COL7 -> COL4
- U1 pad 15: COL8 -> COL3
- U1 pad 16: COL9 -> COL2
- U1 pad 17: COL10 -> COL1
- U1 pad 18: COL11 -> COL0
- U1 pad 7: COL0 -> COL6
- U1 pad 8: COL1 -> COL7
- U1 pad 9: COL2 -> COL8
Routing:
- net COL0: track 537.9 -> 143.0 mm
- net VCC: track 716.5 -> 324.7 mm, vias 3 -> 0
- net GND: track 637.6 -> 255.5 mm, vias 2 -> 0
- net COL1: track 460.2 -> 172.1 mm
- net COL2: track 424.8 -> 159.9 mm
- net ROW7: track 257.4 -> 0.00 mm
- net COL3: track 355.6 -> 149.5 mm
- net ROW6: track 190.5 -> 0.00 mm
- net ROW5: track 168.1 -> 0.00 mm
- net COL4: track 287.1 -> 132.3 mm
- net COL5: track 235.8 -> 87.1 mm
- net ROW4: track 134.1 -> 0.00 mm
- net Net-(LED4-Pad2): track 111.3 -> 0.00 mm
- net ROW3: track 173.1 -> 80.6 mm
- net Net-(LED1-Pad2): track 84.2 -> 0.00 mm
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Other:
- outline, holes or cut-outs redrawn

Commit message: The routing is over jeez
Parts:
- moved LED4 24.2 mm to (212.2, 112.1), turned to 28 degrees
- moved D42 21.7 mm to (171.6, 112.3), turned to 323 degrees
- moved D9 14.0 mm to (183.6, 45.2), turned to 298 degrees
- moved D44 11.0 mm to (188.0, 122.2), turned to 323 degrees
- moved D43 10.6 mm to (175.9, 138.8), turned to 332 degrees
- moved LED2 8.96 mm to (245.9, 43.2), turned to 208 degrees
- moved SW42 4.33 mm to (166.6, 118.9)
- moved D25 3.65 mm to (35.7, 67.9)
- moved J1 3.65 mm to (151.9, 54.3)
- moved D14 3.65 mm to (61.5, 60.0)
- moved D19 3.65 mm to (177.7, 80.1)
- moved D24 3.65 mm to (251.4, 51.0)
- moved D27 3.65 mm to (75.0, 75.2)
- moved D28 3.65 mm to (94.6, 78.9)
- moved D30 3.65 mm to (124.1, 104.6)
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- renumbered Dn to D41
Connections:
- U1 pad 10: COL9 -> COL8
- U1 pad 11: COL10 -> COL7
- U1 pad 12: COL11 -> COL6
- U1 pad 25: ENC1A -> ENC2A
- U1 pad 26: ENC1B -> ENC2B
- U1 pad 28: ENC2A -> ENC1A
- U1 pad 29: ENC2B -> ENC1B
- U1 pad 7: COL6 -> COL11
- U1 pad 8: COL7 -> COL10
- U1 pad 9: COL8 -> COL9
Routing:
- net GND: track 255.5 -> 838.9 mm, vias 0 -> 2
- net VCC: track 324.7 -> 692.6 mm, vias 0 -> 1
- net ROW2: track 107.6 -> 350.7 mm, vias 0 -> 1
- net ROW1: track 107.6 -> 327.3 mm, vias 0 -> 1
- net ROW3: track 80.6 -> 299.4 mm, vias 0 -> 1
- net COL10: track 0.00 -> 168.0 mm
- net ROW0: track 140.9 -> 301.9 mm
- net COL9: track 0.00 -> 150.8 mm
- net COL8: track 0.00 -> 146.6 mm
- net COL11: track 0.00 -> 136.1 mm
- net COL7: track 0.00 -> 128.2 mm
- net ENC1A: track 0.00 -> 111.8 mm
- net ENC1B: track 0.00 -> 102.6 mm
- net ENC2B: track 0.00 -> 100.4 mm
- net ENC2A: track 0.00 -> 89.1 mm
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
Commit message: Move down the left pinky cluster 0.25u
Parts:
- moved D13 4.77 mm to (42.3, 55.2)
- moved D14 4.77 mm to (59.1, 64.1)
- moved MX2 4.77 mm to (60.8, 43.4)
- moved MX1 4.77 mm to (43.9, 34.5)
- moved D25 4.77 mm to (33.3, 72.0)
- moved MX14 4.77 mm to (51.8, 60.2)
- moved MX13 4.77 mm to (35.0, 51.3)
- moved D26 4.77 mm to (50.1, 80.9)
- moved MX26 4.77 mm to (42.9, 77.0)
- moved MX25 4.77 mm to (26.0, 68.1)
- moved D34 0.21 mm to (235.5, 67.4)
- moved D46 0.21 mm to (206.8, 104.8)
- moved D21 0.21 mm to (207.0, 54.2)
- moved D7 0.21 mm to (168.5, 63.1)
- moved LED4 0.21 mm to (212.0, 112.0)
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Routing:
- net ROW2: track 350.7 -> 369.5 mm
- net GND: track 838.9 -> 832.2 mm
- net Net-(LED8-Pad2): track 65.8 -> 60.7 mm
- net COL0: track 143.0 -> 147.7 mm
- net ROW0: track 301.9 -> 305.0 mm
- net COL1: track 172.1 -> 174.9 mm
- net VCC: track 692.6 -> 694.8 mm
- net ROW1: track 327.3 -> 329.4 mm
- net Net-(D25-Pad2): track 6.20 -> 7.25 mm
- net Net-(D2-Pad2): track 6.20 -> 7.19 mm
- net Net-(D1-Pad2): track 6.20 -> 7.19 mm

Commit message: Routing is over
Parts:
- moved D36 4.46 mm to (262.1, 71.8)
- moved MX11 4.46 mm to (234.7, 43.2)
- moved MX35 4.46 mm to (252.6, 76.9)
- moved D23 4.46 mm to (250.9, 56.2)
- moved D24 4.46 mm to (253.2, 55.0)
- moved MX23 4.46 mm to (243.7, 60.0)
- moved MX36 4.46 mm to (269.4, 67.9)
- moved D35 4.46 mm to (259.9, 73.0)
- moved MX24 4.46 mm to (260.5, 51.1)
- moved MX12 4.46 mm to (251.5, 34.3)
- moved LED2 0.33 mm to (245.4, 43.0)
- moved LED3 0.33 mm to (269.1, 80.6)
- moved D40 0.33 mm to (127.5, 153.1)
- moved LED6 0.33 mm to (83.5, 111.8)
- moved MX22 0.33 mm to (219.0, 54.2)
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Routing:
- net COL10: track 168.0 -> 174.9 mm
- net VCC: track 694.8 -> 701.1 mm
- net Net-(LED10-Pad4): track 64.5 -> 70.1 mm
- net COL11: track 136.1 -> 140.8 mm
- net GND: track 832.2 -> 835.1 mm
- net Net-(LED1-Pad2): track 85.4 -> 88.2 mm
- net ROW1: track 329.4 -> 331.4 mm
- net ROW2: track 369.5 -> 371.5 mm
- net ROW0: track 305.0 -> 303.9 mm
- net Net-(D12-Pad2): track 11.3 -> 12.3 mm
- net Net-(D11-Pad2): track 6.20 -> 7.19 mm
- net SDA: track 24.4 -> 25.2 mm
