File: flatbrain.kicad_pcb (KiCad board)
At the start: 2 copper layers, 249.8 x 129.3 mm, 90 parts, among them J1 OLED, J2 Conn_01x05, SW1 Rotary_Encoder_Switch, SW2 Rotary_Encoder_Switch, U1 Elite-C

Commit message: some more silk
Parts:
- moved D14 5.75 mm to (74.8, 99.6)
- moved D15 5.75 mm to (80.1, 102.4)
- moved SW2 5.75 mm to (167.1, 121.2)
- moved D35 5.75 mm to (74.9, 112.2)
- moved MX17 5.75 mm to (192.5, 80.6)
- moved MX30 5.75 mm to (260.6, 86.9)
- moved D30 5.75 mm to (248.1, 100.9)
- moved D9 5.75 mm to (237.7, 94.0)
- moved J2 5.75 mm to (161.9, 111.3)
- moved D33 5.75 mm to (64.3, 106.5)
- moved MX22 5.75 mm to (67.0, 79.1)
- moved D24 5.75 mm to (66.3, 109.3)
- moved MX6 5.75 mm to (167.9, 74.8)
- moved D26 5.75 mm to (232.2, 109.3)
- moved LED6 5.75 mm to (150.9, 153.0)
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Routing:
- net COL2: track 203.2 -> 216.0 mm
- net Net-(D32-Pad2): track 58.7 -> 52.5 mm
- net Net-(D33-Pad2): track 84.4 -> 78.4 mm
- net Net-(D34-Pad2): track 110.3 -> 104.5 mm
- net COL7: track 197.6 -> 202.1 mm
- net COL8: track 210.5 -> 212.4 mm
- net ROW3: track 321.7 -> 323.2 mm
- net Net-(D2-Pad2): track 67.2 -> 65.7 mm
- net Net-(D12-Pad2): track 47.5 -> 46.0 mm
- net GND: track 736.3 -> 737.7 mm
- net ROW1: track 396.1 -> 394.7 mm
- net COL3: track 187.6 -> 188.7 mm
- net ROW0: track 387.8 -> 386.9 mm
- net COL6: track 179.1 -> 180.0 mm
- net ROW2: track 342.8 -> 343.6 mm
Other:
- board text added: "Master can't be dead! Who will tell Thori he's a good dog? Unmurder master now!"
- board text added: "Merging a split board a dumb idea by louckousse"

Commit message: move diode 1.5mm
Parts:
- moved D18 1.47 mm to (231.6, 100.4)
- moved D36 1.47 mm to (228.1, 113.1)
- moved D38 1.47 mm to (236.8, 110.2)
- moved D16 1.47 mm to (221.0, 106.1)
- moved D17 1.47 mm to (226.3, 103.3)
- moved D28 1.47 mm to (244.0, 104.6)
- moved D29 1.47 mm to (247.3, 104.5)
- moved D30 1.47 mm to (249.3, 101.8)
- moved D6 1.47 mm to (222.9, 103.3)
- moved D8 1.47 mm to (233.5, 97.7)
- moved D20 1.47 mm to (242.2, 94.8)
- moved D37 1.47 mm to (242.1, 107.3)
- moved D27 1.47 mm to (238.7, 107.4)
- moved D39 1.47 mm to (231.5, 113.0)
- moved D10 1.47 mm to (244.1, 92.1)
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Routing:
- net Net-(D29-Pad2): track 35.4 -> 38.1 mm
- net ROW2: track 343.6 -> 340.9 mm
- net Net-(D24-Pad2): track 64.3 -> 62.5 mm
- net ROW1: track 394.7 -> 396.5 mm
- net ROW3: track 323.2 -> 321.5 mm
- net Net-(D9-Pad2): track 74.8 -> 76.4 mm
- net Net-(D27-Pad2): track 52.1 -> 53.7 mm
- net Net-(D17-Pad2): track 51.6 -> 53.1 mm
- net Net-(D1-Pad2): track 55.1 -> 56.6 mm
- net Net-(D2-Pad2): track 65.7 -> 67.2 mm
- net Net-(D12-Pad2): track 46.0 -> 47.5 mm
- net Net-(D3-Pad2): track 77.0 -> 78.5 mm
- net Net-(D18-Pad2): track 70.2 -> 71.7 mm
- net Net-(D19-Pad2): track 56.0 -> 57.5 mm
- net Net-(D13-Pad2): track 59.1 -> 60.6 mm
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
Commit message: half pcba
Parts:
- removed G***: LOGO, cc:cc
- added C1: 1uF, Capacitor_SMD:C_0805_2012Metric, F.Cu at (138.1, 92.8)
- added C2: 0.1uF, Capacitor_SMD:C_0805_2012Metric, F.Cu at (135.2, 104.5)
- added C3: 0.1uF, Capacitor_SMD:C_0805_2012Metric, F.Cu at (148.9, 90.9)
- added C4: 0.1uF, Capacitor_SMD:C_0805_2012Metric, F.Cu at (154.2, 96.2)
- added C5: 10uF, Capacitor_SMD:C_0805_2012Metric, F.Cu at (146.3, 88.3)
- added C6: 22pF, Capacitor_SMD:C_0805_2012Metric, F.Cu at (136.5, 111.4)
- added C7: 22pF, Capacitor_SMD:C_0805_2012Metric, F.Cu at (134.3, 109.3)
- added C8: 0.1uF, Capacitor_SMD:C_0805_2012Metric, F.Cu at (148.6, 109.6)
- added F1: 500mA, Fuse:Fuse_1206_3216Metric, F.Cu at (150.1, 43.9)
- added FB1: Ferrite_Bead_Small, Inductor_SMD:L_0805_2012Metric_Pad1.15x1.40mm_HandSolder, F.Cu at (138.1, 34.0)
- added J3: AVR-ISP-6, random-keyboard-parts:Reset_Pretty-Mask, B.Cu at (137.3, 52.2)
- added R1: 10k, Resistor_SMD:R_0805_2012Metric, F.Cu at (156.1, 100.4)
- added R2: 22, Resistor_SMD:R_0805_2012Metric, F.Cu at (142.6, 87.4)
- added R3: 22, Resistor_SMD:R_0805_2012Metric, F.Cu at (140.6, 87.4)
- added R4: 10k, Resistor_SMD:R_0805_2012Metric, F.Cu at (137.7, 56.3)
- added R5: 5.1k, Resistor_SMD:R_0805_2012Metric, F.Cu at (149.9, 38.2)
- added R6: 5.1k, Resistor_SMD:R_0805_2012Metric, F.Cu at (139.9, 38.2)
- added SW3: SW_Push, random-keyboard-parts:SKQG-1155865, F.Cu at (145.3, 69.2)
- added U2: PRTR5V0U2X, random-keyboard-parts:SOT143B, F.Cu at (145.5, 42.2)
- added USB1: USB_C_Receptacle_USB2.0, Connector_USB:USB_C_Receptacle_HRO_TYPE-C-31-M-12, F.Cu at (145.5, 30.6)
- added Y1: 16MHz, Crystal:Crystal_SMD_3225-4Pin_3.2x2.5mm, F.Cu at (138.2, 107.5)
- U1: value Elite-C -> ATmega32U4-AU; footprint Keebio-Parts:Elite-C -> Package_QFP:TQFP-44_10x10mm_P0.8mm; moved to F.Cu
- moved U1 55.0 mm to (145.3, 100.4), turned to 315 degrees
- moved D3 7.05 mm to (65.1, 104.0)
- moved D16 7.05 mm to (214.9, 109.6)
- moved SW2 7.05 mm to (161.5, 124.3)
- moved LED10 7.05 mm to (95.3, 36.3)
- moved LED2 7.05 mm to (195.3, 36.3)
- moved D32 7.05 mm to (63.3, 113.8)
- moved D39 7.05 mm to (225.4, 116.5)
- moved MX17 7.05 mm to (186.9, 83.7)
- moved MX20 7.05 mm to (246.1, 73.3)
- moved D21 7.05 mm to (47.4, 105.4)
- moved MX22 7.05 mm to (61.4, 82.2)
- moved D19 7.05 mm to (230.8, 101.2)
- moved D25 7.05 mm to (65.3, 116.5)
- moved D5 7.05 mm to (75.7, 109.6)
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Connections:
- J1 pad 3: VCC -> +5V
- J2 pad 1: VCC -> +5V
- LED1 pad 1: VCC -> +5V
- LED10 pad 1: VCC -> +5V
- LED2 pad 1: VCC -> +5V
- LED3 pad 1: VCC -> +5V
- LED4 pad 1: VCC -> +5V
- LED5 pad 1: VCC -> +5V
- LED6 pad 1: VCC -> +5V
- LED7 pad 1: VCC -> +5V
- LED8 pad 1: VCC -> +5V
- LED9 pad 1: VCC -> +5V
- U1 pad 10: COL5 -> COL2
- U1 pad 11: ROW2 -> COL3
- U1 pad 12: ROW3 -> COL4
- U1 pad 13: Net-(U1-Pad13) -> RST
- U1 pad 14: ROW1 -> +5V
- U1 pad 15: ROW0 -> GND
- U1 pad 16: COL4 -> XTAL2
- U1 pad 17: COL3 -> XTAL1
- U1 pad 18: COL2 -> SCL
- U1 pad 19: COL1 -> SDA
- U1 pad 2: COL9 -> +5V
- U1 pad 20: COL0 -> COL5
- U1 pad 21: VCC -> ENC1A
- U1 pad 22: Net-(U1-Pad22) -> ENC1B
- U1 pad 24: Net-(U1-Pad24) -> +5V
- U1 pad 25: ENC2A -> COL7
- U1 pad 26: ENC2B -> ROW3
- U1 pad 27: Net-(U1-Pad27) -> ROW2
- U1 pad 28: ENC1B -> ROW0
- U1 pad 29: ENC1A -> COL6
- U1 pad 3: GND -> D-
- U1 pad 4: GND -> D+
- U1 pad 5: SDA -> GND
- U1 pad 6: SCL -> Net-(C1-Pad1)
- U1 pad 7: COL8 -> +5V
- U1 pad 8: COL7 -> COL0
- U1 pad 9: COL6 -> COL1
Routing:
- net +5V: track 0.00 -> 761.7 mm, vias 0 -> 6
- net VCC: track 679.2 -> 19.8 mm
- net COL1: track 220.3 -> 383.3 mm
- net COL0: track 180.6 -> 291.4 mm
- net COL2: track 216.0 -> 324.9 mm
- net ROW2: track 340.9 -> 236.9 mm, vias 1 -> 0
- net ROW3: track 321.5 -> 220.3 mm, vias 1 -> 0
- net ROW1: track 396.5 -> 306.6 mm, vias 1 -> 0
- net COL3: track 188.7 -> 278.2 mm
- net COL9: track 176.1 -> 89.2 mm
- net Net-(D24-Pad2): track 62.5 -> 147.9 mm
- net ROW0: track 385.6 -> 304.5 mm, vias 1 -> 0
- net ENC2A: track 80.9 -> 0.00 mm
- net ENC2B: track 74.6 -> 0.00 mm
- net GND: track 737.7 -> 809.6 mm, vias 0 -> 3
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- added copper zone on B.Cu, net Earth
- added copper zone on F.Cu, net Earth
- added copper zone on F.Cu, net GND
Other:
- board size 249.8 x 129.3 mm -> 249.8 x 132.9 mm

Commit message: pcba over
Parts:
- moved C4 5.81 mm to (160.0, 95.3)
- moved USB1 5.55 mm to (150.9, 29.2)
- moved D34 5.54 mm to (58.1, 106.9)
- moved J1 5.54 mm to (146.9, 60.1)
- moved LED2 5.54 mm to (200.7, 35.0)
- moved D1 5.54 mm to (59.9, 97.1)
- moved MX21 5.54 mm to (41.0, 88.8)
- moved D15 5.54 mm to (79.2, 105.6)
- moved MX6 5.54 mm to (167.7, 76.7)
- moved D19 5.54 mm to (236.2, 99.9)
- moved MX10 5.54 mm to (242.5, 55.1)
- moved MX24 5.54 mm to (100.2, 99.2)
- moved MX25 5.54 mm to (115.8, 110.3)
- moved D17 5.54 mm to (225.6, 105.5)
- moved MX16 5.54 mm to (176.6, 93.5)
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Connections:
- U1 pad 20: COL5 -> Net-(U1-Pad20)
- U1 pad 25: COL7 -> Net-(U1-Pad25)
- U1 pad 26: ROW3 -> Net-(U1-Pad26)
- U1 pad 27: ROW2 -> ROW1
- U1 pad 29: COL6 -> ROW3
- U1 pad 30: ROW1 -> ROW2
- U1 pad 37: Net-(U1-Pad37) -> COL5
- U1 pad 38: COL9 -> COL6
- U1 pad 39: COL8 -> COL7
- U1 pad 40: Net-(U1-Pad40) -> COL8
- U1 pad 41: Net-(U1-Pad41) -> COL9
Routing:
- net ROW2: track 236.9 -> 412.2 mm, vias 0 -> 1
- net ROW1: track 306.6 -> 474.8 mm
- net ROW3: track 220.3 -> 388.5 mm, vias 0 -> 1
- net COL9: track 89.2 -> 192.1 mm
- net COL8: track 151.8 -> 241.1 mm
- net COL0: track 291.4 -> 202.5 mm
- net SCL: track 19.2 -> 93.7 mm, vias 0 -> 1
- net SDA: track 19.4 -> 91.7 mm, vias 0 -> 1
- net COL1: track 383.3 -> 318.9 mm
- net ENC2B: track 0.00 -> 62.1 mm
- net COL7: track 159.0 -> 217.6 mm
- net ENC2A: track 0.00 -> 56.3 mm
- net Net-(D19-Pad2): track 57.5 -> 105.0 mm
- net COL6: track 155.2 -> 202.0 mm
- net COL2: track 324.9 -> 279.0 mm
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Other:
- board size 249.8 x 132.9 mm -> 249.8 x 133.4 mm

Commit message: edge cuts
Parts:
- moved USB1 0.22 mm to (150.7, 29.2)
Other:
- board size 249.8 x 133.4 mm -> 249.8 x 133.3 mm

Commit message: ready to prod
Parts:
- added G***: LOGO, cc:cc, F.Cu at (150.9, 51.1)
- renumbered SW3 to RST1, J2 to trackball
Routing:
- net COL4: track 141.8 -> 144.4 mm
- net ROW2: track 412.2 -> 409.8 mm
- net RST: track 68.6 -> 70.9 mm
- net COL5: track 147.0 -> 145.9 mm
- net GND: track 819.1 -> 818.6 mm, vias 3 -> 4
- net +5V: track 762.4 -> 762.3 mm, vias 6 -> 7
- added copper zone on B.Cu, net GND

Commit message: move thumb cluster
Parts:
- moved G*** 6.37 mm to (150.4, 44.7)
- moved MX33 1.91 mm to (114.8, 133.2)
- moved MX38 1.91 mm to (186.6, 133.2)
- moved MX34 1.76 mm to (130.1, 146.8), turned to 313.8 degrees
- moved MX37 1.75 mm to (171.3, 146.8), turned to 46.2 degrees
- moved MX39 1.12 mm to (203.9, 122.1), turned to 28 degrees
- moved MX32 1.11 mm to (97.5, 122.1), turned to 332 degrees
Routing:
- net Net-(D32-Pad2): track 53.7 -> 60.5 mm
- net Net-(D33-Pad2): track 78.4 -> 85.2 mm
- net Net-(D38-Pad2): track 59.7 -> 64.9 mm
- net COL2: track 278.6 -> 281.3 mm
- net COL1: track 318.9 -> 316.3 mm
- net COL6: track 202.0 -> 204.5 mm
- net +5V: track 762.3 -> 764.1 mm
- net COL8: track 241.1 -> 239.5 mm
- net Net-(D39-Pad2): track 32.1 -> 30.7 mm
- net GND: track 818.6 -> 819.8 mm
- net COL3: track 265.2 -> 266.2 mm
- net Net-(LED6-Pad2): track 47.8 -> 48.6 mm

Commit message: routing
Routing:
- net COL3: track 266.2 -> 256.6 mm
- net ENC2A: track 56.3 -> 50.3 mm
- net ENC2B: track 62.1 -> 57.1 mm
- net COL6: track 204.5 -> 202.4 mm
- net RST: track 70.9 -> 68.9 mm
- net SDA: track 91.7 -> 93.6 mm
- net COL4: track 144.4 -> 146.0 mm
- net SCL: track 93.7 -> 94.7 mm
- net COL8: track 239.5 -> 238.7 mm
- net COL1: track 316.3 -> 316.9 mm
