File: pcb/flatbrain.kicad_pcb (KiCad board)
At the start: 2 copper layers, 272.2 x 143 mm, 101 parts, among them J1 OLED, SW1 SW_Push, U1 kbd_ProMicro

Commit message: Move all files between two folder
PCB: contains everything pcb related
CASE: contains everythind dxf related or non electronical
Parts:
- moved MX31 0.23 mm to (179.0, 100.9)
- moved MX6 0.23 mm to (134.4, 67.2)
- moved D3 0.23 mm to (81.3, 44.4)
- moved MX28 0.23 mm to (87.0, 75.1)
- moved MX29 0.23 mm to (100.8, 89.8)
- moved D12 0.23 mm to (252.0, 34.8)
- moved MX10 0.23 mm to (210.2, 37.8)
- moved D31 0.23 mm to (186.0, 97.2)
- moved D42 0.23 mm to (183.7, 130.7)
- moved MX8 0.23 mm to (176.8, 56.2)
- moved D16 0.23 mm to (103.1, 61.1)
- moved D27 0.23 mm to (74.3, 75.2)
- moved D39 0.23 mm to (123.0, 129.9)
- moved MX25 0.23 mm to (28.1, 64.1)
- moved MX26 0.23 mm to (45.0, 73.1)
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