File: case/bottom/bottom.kicad_pcb (KiCad board)
At the start: 2 copper layers, 272.2 x 143 mm, 9 parts

Commit message: Update the outline with the new design
Parts:
- removed REF** (x9): MountingHole_2.2mm_M2_Pad, MountingHole:MountingHole_2.2mm_M2_Pad
Routing:
- removed copper zone on B.Cu, net (none)
- removed copper zone on F.Cu, net (none)
Other:
- board size 272.2 x 143 mm -> 268.7 x 141.1 mm
- board text removed: "JLCJLCJLCJLC"
- board text removed: "UP HERE"
