File: case/plate/plate.kicad_pcb (KiCad board)
At the start: 2 copper layers, 272.2 x 143.4 mm, 9 parts

Commit message: Correct the size of the switch hole
Parts:
- removed the REF** at (275.8, 87.6)
- removed the REF** at (219.7, 104.3)
- removed the REF** at (147.2, 135.5)
- removed the REF** at (74.7, 104.3)
- removed the REF** at (18.7, 87.6)
- removed the REF** at (70.2, 34.8)
- removed the REF** at (127.8, 44.2)
- removed the REF** at (166.6, 44.2)
- added REF**: MountingHole_2.2mm_M2_Pad, MountingHole:MountingHole_2.2mm_M2_Pad, F.Cu at (278.1, 77.8)
- added REF**: MountingHole_2.2mm_M2_Pad, MountingHole:MountingHole_2.2mm_M2_Pad, F.Cu at (222.1, 94.5)
- added REF**: MountingHole_2.2mm_M2_Pad, MountingHole:MountingHole_2.2mm_M2_Pad, F.Cu at (149.6, 125.7)
- added REF**: MountingHole_2.2mm_M2_Pad, MountingHole:MountingHole_2.2mm_M2_Pad, F.Cu at (77.1, 94.5)
- added REF**: MountingHole_2.2mm_M2_Pad, MountingHole:MountingHole_2.2mm_M2_Pad, F.Cu at (21.0, 77.8)
- added REF**: MountingHole_2.2mm_M2_Pad, MountingHole:MountingHole_2.2mm_M2_Pad, F.Cu at (72.6, 25.0)
- added REF**: MountingHole_2.2mm_M2_Pad, MountingHole:MountingHole_2.2mm_M2_Pad, F.Cu at (130.2, 34.4)
- added REF**: MountingHole_2.2mm_M2_Pad, MountingHole:MountingHole_2.2mm_M2_Pad, F.Cu at (169.0, 34.4)
- moved REF** 10.1 mm to (226.5, 25.0)
Other:
- outline, holes or cut-outs redrawn

Commit message: Update the outline with the new design
Parts:
- removed REF** (x9): MountingHole_2.2mm_M2_Pad, MountingHole:MountingHole_2.2mm_M2_Pad
Other:
- board size 272.2 x 143.4 mm -> 268.7 x 136.6 mm
- board text removed: "designed by louckousse"
